Commit message: ros2: description, display launch, transient robot_description publisher, control scaffold

File: ros2/handy_description/urdf/handy_description.urdf.xacro (robot description, xacro)
@@ -491,3 +491,53 @@
     <xacro:transmission name="tran9" joint="joint_9" actuator="motor_9" />
   </xacro:if>
+  <ros2_control name="HandySystem" type="system">
+    <hardware>
+      <plugin>mock_components/GenericSystem</plugin>
+    </hardware>
+    <joint name="joint_1">
+      <command_interface name="position"/>
+      <state_interface name="position"/>
+      <state_interface name="velocity"/>
+    </joint>
+    <joint name="joint_2">
+      <command_interface name="position"/>
+      <state_interface name="position"/>
+      <state_interface name="velocity"/>
+    </joint>
+    <joint name="joint_3">
+      <command_interface name="position"/>
+      <state_interface name="position"/>
+      <state_interface name="velocity"/>
+    </joint>
+    <joint name="joint_4">
+      <command_interface name="position"/>
+      <state_interface name="position"/>
+      <state_interface name="velocity"/>
+    </joint>
+    <joint name="joint_5">
+      <command_interface name="position"/>
+      <state_interface name="position"/>
+      <state_interface name="velocity"/>
+    </joint>
+    <joint name="joint_6">
+      <command_interface name="position"/>
+      <state_interface name="position"/>
+      <state_interface name="velocity"/>
+    </joint>
+    <joint name="joint_7">
+      <command_interface name="position"/>
+      <state_interface name="position"/>
+      <state_interface name="velocity"/>
+    </joint>
+    <joint name="joint_8">
+      <command_interface name="position"/>
+      <state_interface name="position"/>
+      <state_interface name="velocity"/>
+    </joint>
+    <joint name="joint_9">
+      <command_interface name="position"/>
+      <state_interface name="position"/>
+      <state_interface name="velocity"/>
+    </joint>
+  </ros2_control>
 </robot>

Commit message: Added hand and arm groups to rviz

File: ros2/handy_description/urdf/handy_description.urdf.xacro (robot description, xacro)
@@ -79,8 +79,8 @@
       <inertia
         ixx="0.00096626194"
-        ixy="-0.00000006431"
-        ixz="0.00000032990"
+        ixy="0.00000000000"
+        ixz="0.00000000000"
         iyy="0.00575735994"
-        iyz="-0.00039309867"
+        iyz="0.00000000000"
         izz="0.00066079574"
       />
@@ -119,8 +119,8 @@
       <inertia
         ixx="0.00067487030"
-        ixy="-0.00005184685"
-        ixz="-0.00000255096"
+        ixy="0.00000000000"
+        ixz="0.00000000000"
         iyy="0.00024791507"
-        iyz="0.00002448920"
+        iyz="0.00000000000"
         izz="0.000052259169"
       />
@@ -420,4 +420,5 @@
   </link>
   <joint name="joint_9" type="revolute">
+    <mimic joint="joint_8" multiplier="-1.0" offset="0.0" />
     <origin xyz="0.0186 0 -0.056505" rpy="1.5708 1.5708 0" />
     <parent link="link_8" />
@@ -489,5 +490,5 @@
     <xacro:transmission name="tran7" joint="joint_7" actuator="motor_7" />
     <xacro:transmission name="tran8" joint="joint_8" actuator="motor_8" />
-    <xacro:transmission name="tran9" joint="joint_9" actuator="motor_9" />
+    <!-- <xacro:transmission name="tran9" joint="joint_9" actuator="motor_9" /> -->
   </xacro:if>
   <ros2_control name="HandySystem" type="system">
@@ -536,5 +537,4 @@
     </joint>
     <joint name="joint_9">
-      <command_interface name="position"/>
       <state_interface name="position"/>
       <state_interface name="velocity"/>

File: ros2/handy_moveit_config/config/handy_description.ros2_control.xacro (robot description, xacro)
@@ -8,4 +8,11 @@
                 <plugin>mock_components/GenericSystem</plugin>
             </hardware>
+            <joint name="joint_8">
+                <command_interface name="position"/>
+                <state_interface name="position">
+                  <param name="initial_value">${initial_positions['joint_8']}</param>
+                </state_interface>
+                <state_interface name="velocity"/>
+            </joint>
             <joint name="joint_1">
                 <command_interface name="position"/>
@@ -36,4 +43,25 @@
                 <state_interface name="velocity"/>
             </joint>
+            <joint name="joint_5">
+                <command_interface name="position"/>
+                <state_interface name="position">
+                  <param name="initial_value">${initial_positions['joint_5']}</param>
+                </state_interface>
+                <state_interface name="velocity"/>
+            </joint>
+            <joint name="joint_6">
+                <command_interface name="position"/>
+                <state_interface name="position">
+                  <param name="initial_value">${initial_positions['joint_6']}</param>
+                </state_interface>
+                <state_interface name="velocity"/>
+            </joint>
+            <joint name="joint_7">
+                <command_interface name="position"/>
+                <state_interface name="position">
+                  <param name="initial_value">${initial_positions['joint_7']}</param>
+                </state_interface>
+                <state_interface name="velocity"/>
+            </joint>
         </ros2_control>
     </xacro:macro>

Commit message: Diagnosing miscommunication between Dynamixel motors and the world.

File: ros2/handy_description/urdf/handy_description.urdf.xacro (robot description, xacro)
@@ -79,8 +79,8 @@
       <inertia
         ixx="0.00096626194"
-        ixy="0.00000000000"
-        ixz="0.00000000000"
+        ixy="-0.00000006431"
+        ixz="0.00000032990"
         iyy="0.00575735994"
-        iyz="0.00000000000"
+        iyz="-0.00039309867"
         izz="0.00066079574"
       />
@@ -119,8 +119,8 @@
       <inertia
         ixx="0.00067487030"
-        ixy="0.00000000000"
-        ixz="0.00000000000"
+        ixy="-0.00005184685"
+        ixz="-0.00000255096"
         iyy="0.00024791507"
-        iyz="0.00000000000"
+        iyz="0.00002448920"
         izz="0.000052259169"
       />
@@ -490,10 +490,91 @@
     <xacro:transmission name="tran7" joint="joint_7" actuator="motor_7" />
     <xacro:transmission name="tran8" joint="joint_8" actuator="motor_8" />
-    <!-- <xacro:transmission name="tran9" joint="joint_9" actuator="motor_9" /> -->
+    <xacro:transmission name="tran9" joint="joint_9" actuator="motor_9" /> <!-- consider removing -->
   </xacro:if>
   <ros2_control name="HandySystem" type="system">
     <hardware>
-      <plugin>mock_components/GenericSystem</plugin>
+      <plugin>dynamixel_hardware_interface/DynamixelHardware</plugin>
+      <param name="port_name">/dev/ttyUSB0</param>
+      <param name="baud_rate">1000000</param>
+      <param name="number_of_joints">9</param>
+      <param name="number_of_transmissions">0</param>
+      <param name="dynamixel_model_folder">/param/dxl_model</param>
+      <param name="disable_torque_at_init">false</param>
+      <param name="protocol_version">1.0</param>
+      <param name="ids">1, 2, 3, 4, 5, 6, 7, 8, 9</param>
+      <param name="joint_names">joint_1, joint_2, joint_3, joint_4, joint_5, joint_6, joint_7, joint_8, joint_9</param>
     </hardware>
+    <gpio name="dxl1">
+      <param name="type">dxl</param>
+      <param name="ID">1</param>
+      <command_interface name="Goal Position"/>
+      <state_interface name="Present Position"/>
+      <state_interface name="Present Velocity"/>
+      <state_interface name="Present Current"/>
+    </gpio>
+    <gpio name="dxl2">
+      <param name="type">dxl</param>
+      <param name="ID">2</param>
+      <command_interface name="Goal Position"/>
+      <state_interface name="Present Position"/>
+      <state_interface name="Present Velocity"/>
+      <state_interface name="Present Current"/>
+    </gpio>
+    <gpio name="dxl3">
+      <param name="type">dxl</param>
+      <param name="ID">3</param>
+      <command_interface name="Goal Position"/>
+      <state_interface name="Present Position"/>
+      <state_interface name="Present Velocity"/>
+      <state_interface name="Present Current"/>
+    </gpio>
+    <gpio name="dxl4">
+      <param name="type">dxl</param>
+      <param name="ID">4</param>
+      <command_interface name="Goal Position"/>
+      <state_interface name="Present Position"/>
+      <state_interface name="Present Velocity"/>
+      <state_interface name="Present Current"/>
+    </gpio>
+    <gpio name="dxl5">
+      <param name="type">dxl</param>
+      <param name="ID">5</param>
+      <command_interface name="Goal Position"/>
+      <state_interface name="Present Position"/>
+      <state_interface name="Present Velocity"/>
+      <state_interface name="Present Current"/>
+    </gpio>
+    <gpio name="dxl6">
+      <param name="type">dxl</param>
+      <param name="ID">6</param>
+      <command_interface name="Goal Position"/>
+      <state_interface name="Present Position"/>
+      <state_interface name="Present Velocity"/>
+      <state_interface name="Present Current"/>
+    </gpio>
+    <gpio name="dxl7">
+      <param name="type">dxl</param>
+      <param name="ID">7</param>
+      <command_interface name="Goal Position"/>
+      <state_interface name="Present Position"/>
+      <state_interface name="Present Velocity"/>
+      <state_interface name="Present Current"/>
+    </gpio>
+    <gpio name="dxl8">
+      <param name="type">dxl</param>
+      <param name="ID">8</param>
+      <command_interface name="Goal Position"/>
+      <state_interface name="Present Position"/>
+      <state_interface name="Present Velocity"/>
+      <state_interface name="Present Current"/>
+    </gpio>
+    <gpio name="dxl9">
+      <param name="type">dxl</param>
+      <param name="ID">9</param>
+      <command_interface name="Goal Position"/>
+      <state_interface name="Present Position"/>
+      <state_interface name="Present Velocity"/>
+      <state_interface name="Present Current"/>
+    </gpio>
     <joint name="joint_1">
       <command_interface name="position"/>
@@ -537,4 +618,5 @@
     </joint>
     <joint name="joint_9">
+      <command_interface name="position"/>
       <state_interface name="position"/>
       <state_interface name="velocity"/>

File: ros2/handy_moveit_config/config/handy_description.ros2_control.xacro (robot description, xacro)
@@ -4,16 +4,26 @@
         <xacro:property name="initial_positions" value="${load_yaml(initial_positions_file)['initial_positions']}"/>
         <ros2_control name="${name}" type="system">
+            <!-- May change later
+            <param name="dynamixel_state_pub_msg_name">dynamixel_hardware_interface/dxl_state</param>
+            <param name="get_dynamixel_data_srv_name">dynamixel_hardware_interface/get_dxl_data</param>
+            <param name="set_dynamixel_data_srv_name">dynamixel_hardware_interface/set_dxl_data</param>
+            <param name="reboot_dxl_srv_name">dynamixel_hardware_interface/reboot_dxl</param>
+            <param name="set_dxl_torque_srv_name">dynamixel_hardware_interface/set_dxl_torque</param>
+            -->
             <hardware>
-                <!-- By default, set up controllers for simulation. This won't work on real hardware -->
-                <plugin>mock_components/GenericSystem</plugin>
+                <plugin>dynamixel_hardware_interface/DynamixelHardware</plugin>
+                <param name="port_name">/dev/ttyUSB0</param>
+                <param name="baud_rate">1000000</param>
+                <param name="number_of_joints">9</param>
+                <param name="number_of_transmissions">0</param>
+                <param name="dynamixel_model_folder">/param/dxl_model</param>
+                <param name="disable_torque_at_init">false</param>
+                <param name="protocol_version">1.0</param>
+                <param name="ids">1, 2, 3, 4, 5, 6, 7, 8, 9</param>
+                <param name="joint_names">joint_1, joint_2, joint_3, joint_4, joint_5, joint_6, joint_7, joint_8, joint_9</param>
             </hardware>
-            <joint name="joint_8">
-                <command_interface name="position"/>
-                <state_interface name="position">
-                  <param name="initial_value">${initial_positions['joint_8']}</param>
-                </state_interface>
-                <state_interface name="velocity"/>
-            </joint>
             <joint name="joint_1">
+                <param name="id">1</param>
+                <param name="motor_type">ex_106</param>
                 <command_interface name="position"/>
                 <state_interface name="position">
@@ -23,4 +33,6 @@
             </joint>
             <joint name="joint_2">
+                <param name="id">2</param>
+                <param name="motor_type">mx_106</param>
                 <command_interface name="position"/>
                 <state_interface name="position">
@@ -30,4 +42,6 @@
             </joint>
             <joint name="joint_3">
+                <param name="id">3</param>
+                <param name="motor_type">ex_106</param>
                 <command_interface name="position"/>
                 <state_interface name="position">
@@ -37,4 +51,6 @@
             </joint>
             <joint name="joint_4">
+                <param name="id">4</param>
+                <param name="motor_type">ex_106</param>
                 <command_interface name="position"/>
                 <state_interface name="position">
@@ -44,4 +60,6 @@
             </joint>
             <joint name="joint_5">
+                <param name="id">5</param>
+                <param name="motor_type">mx_28</param>
                 <command_interface name="position"/>
                 <state_interface name="position">
@@ -51,4 +69,6 @@
             </joint>
             <joint name="joint_6">
+                <param name="id">6</param>
+                <param name="motor_type">mx_28</param>
                 <command_interface name="position"/>
                 <state_interface name="position">
@@ -58,4 +78,6 @@
             </joint>
             <joint name="joint_7">
+                <param name="id">7</param>
+                <param name="motor_type">mx_28</param>
                 <command_interface name="position"/>
                 <state_interface name="position">
@@ -64,4 +86,22 @@
                 <state_interface name="velocity"/>
             </joint>
+            <joint name="joint_8">
+                <param name="id">8</param>
+                <param name="motor_type">ax_12a</param>
+                <command_interface name="position"/>
+                <state_interface name="position">
+                  <param name="initial_value">${initial_positions['joint_8']}</param>
+                </state_interface>
+                <state_interface name="velocity"/>
+            </joint>
+            <joint name="joint_9">
+                <param name="id">9</param>
+                <param name="motor_type">ax_12a</param>
+                <command_interface name="position"/>
+                <state_interface name="position">
+                  <param name="initial_value">${initial_positions['joint_9']}</param>
+                </state_interface>
+                <state_interface name="velocity"/>
+            </joint>
         </ros2_control>
     </xacro:macro>
